File: EE330_FinalProject/EE330_FinalProject.kicad_sch (KiCad schematic)
At the start: 7 parts, among them IC1 LT1490AIS8#PBF, Q1 2N3904, Q2 2N3904

Commit message: Worked on schematic added astable multivibrator, mounting holes and connector
Parts:
- added C1: 40u4, symbol Device:C_Polarized
- added C2: 17u3, symbol Device:C_Polarized
- added H1, H2, H3, H4: PT, MountingHole:MountingHole_3.2mm_M3_DIN965_Pad_TopBottom, symbol Mechanical:MountingHole_Pad
- added J1: 01x04_Pin, symbol Connector:Conn_01x04_Pin
- added Q3, Q4: 2N3904, Package_TO_SOT_THT:TO-92_Inline, symbol Transistor_BJT:2N3904
- added R5, R7: 4k7, symbol Device:R
- added R6, R8: 100k, symbol Device:R
- R1, R2, R3, R4: value R -> 10k
Connections:
- net Battery: now also J1.1 (Pin_1)
- net GND: now also H1.1, H2.1, H3.1, H4.1, J1.2 (Pin_2), J1.4 (Pin_4), Q3.1 (E), Q4.1 (E)
- net Oscillator: now also R5.1, R6.1, R7.1, R8.1
- net SolarPanel: now also J1.3 (Pin_3)
- new net: C2.1, Q4.3 (C), R7.2
- new net LED_OUT: C1.1, Q3.3 (C), R5.2
- new net N1: C1.2, Q3.2 (B), R6.2
- new net N2: C2.2, Q4.2 (B), R8.2
Other:
- note added: "Astable Multivibrator Oscillator"
- note added: "Mounting Holes and Connector"

Commit message: Updated PCB with component footprints and started Board design
Parts:
- C1, C2: footprint (none) -> Capacitor_SMD:C_0805_2012Metric
- J1: footprint (none) -> Connector_PinHeader_1.27mm:PinHeader_1x04_P1.27mm_Vertical
- R1, R2, R3, R4, R5, R6, R7, R8: footprint (none) -> Resistor_SMD:R_0603_1608Metric
Other:
- note added: "This will probably be a 50uF and a 10uF caps"
Changed lines of the file:
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@@
+		)
+	)
+	(text "This will probably be a 50uF and a 10uF caps"
+		(exclude_from_sim no)
+		(at 252.222 61.468 0)
+		(effects
+			(font
+				(size 1.27 1.27)
+			)
 		)
 	)
@@
 			)
 		)
-		(property "Footprint" ""
+		(property "Footprint" "Resistor_SMD:R_0603_1608Metric"
 			(at 78.74 65.278 90)
 			(effects
@@
 			)
 		)
-		(property "Footprint" ""
+		(property "Footprint" "Capacitor_SMD:C_0805_2012Metric"
 			(at 181.61 61.9252 0)
 			(effects
@@
 			)
 		)
-		(property "Footprint" ""
+		(property "Footprint" "Resistor_SMD:R_0603_1608Metric"
 			(at 46.99 70.358 90)
 			(effects
@@
 			)
 		)
-		(property "Footprint" ""
+		(property "Footprint" "Resistor_SMD:R_0603_1608Metric"
 			(at 149.352 52.07 90)
 			(effects
@@
 			)
 		)
-		(property "Footprint" ""
+		(property "Footprint" "Resistor_SMD:R_0603_1608Metric"
 			(at 61.722 50.8 90)
 			(effects
@@
 			)
 		)
-		(property "Footprint" ""
+		(property "Footprint" "Resistor_SMD:R_0603_1608Metric"
 			(at 90.932 50.8 90)
 			(effects
@@
 			)
 		)
-		(property "Footprint" ""
+		(property "Footprint" "Connector_PinHeader_1.27mm:PinHeader_1x04_P1.27mm_Vertical"
 			(at 167.64 96.52 0)
 			(effects
@@
 			)
 		)
-		(property "Footprint" ""
+		(property "Footprint" "Capacitor_SMD:C_0805_2012Metric"
 			(at 166.37 59.9948 0)
 			(effects
@@
 			)
 		)
-		(property "Footprint" ""
+		(property "Footprint" "Resistor_SMD:R_0603_1608Metric"
 			(at 195.072 52.07 90)
 			(effects
@@
 			)
 		)
-		(property "Footprint" ""
+		(property "Footprint" "Resistor_SMD:R_0603_1608Metric"
 			(at 136.652 52.07 90)
 			(effects
@@
 			)
 		)
-		(property "Footprint" ""
+		(property "Footprint" "Resistor_SMD:R_0603_1608Metric"
 			(at 207.772 52.07 90)
 			(effects
